Commit message: Added lidar obstacle avoidance

File: src/my_bot/description/gazebo_control.xacro (robot description, xacro)
@@ -1,3 +1,18 @@
 <?xml version="1.0"?>
 <robot xmlns:xacro="http://www.ros.org/wiki/xacro">
+<gazebo>
+  <plugin name="diff_drive" filename="libgazebo_ros_diff_drive.so">
+        <left_joint>left_wheel_joint</left_joint>
+        <right_joint>right_wheel_joint</right_joint>
+        <wheel_separation>0.35</wheel_separation>
+        <wheel_diameter>0.1</wheel_diameter>
+        <max_wheel_torque>200</max_wheel_torque>
+        <max_wheel_acceleration>10.0</max_wheel_acceleration>
+        <odometry_frame>odom</odometry_frame>
+        <robot_base_frame>base_link</robot_base_frame>
+        <publish_odom>true</publish_odom>
+        <publish_odom_tf>true</publish_odom_tf>
+        <publish_wheel_tf>true</publish_wheel_tf>
+    </plugin>
+    </gazebo>
 </robot>

File: src/my_bot/description/robot.urdf.xacro (robot description, xacro)
@@ -3,4 +3,6 @@
    <xacro:include filename="$(find my_bot)/description/robot_core.xacro" />
    <xacro:include filename="$(find my_bot)/description/gazebo_control.xacro"/>
-<xacro:include filename="$(find my_bot)/description/lidar.xacro"/>
+    <xacro:include filename="$(find my_bot)/description/lidar.xacro"/>
+   <!-- <xacro:include filename="$(find my_bot)/description/camera.xacro"/> -->
+     <xacro:include filename="$(find my_bot)/description/depth_camera.xacro"/>
 </robot>

File: src/my_bot/description/robot_core.xacro (robot description, xacro)
@@ -122,3 +122,8 @@
               </xacro:inertial_sphere>
      </link>
+     <gazebo reference="caster_wheel">
+       <material>Gazebo/Black</material>
+       <mu1 value="0.001"/>
+       <mu2 value="0.001"/>
+       </gazebo>
 </robot>
